Commit message: Added conveyor and refactored world

File: MOBILE_MANIPULATOR/mobile_manipulator_description/urdf/camera_module.urdf.xacro (robot description, xacro)
@@ -4,7 +4,7 @@
     <link name="camera_link_base">
       <visual>
-        <origin xyz="0 0 0" rpy="0 0 1.57"/>
+        <origin xyz="0 0 0" rpy="1.57 3.14 1.57"/>
         <geometry>
-          <mesh filename="$(find mobile_manipulator_description)/meshes/realsense.dae" scale="1 1 1"/>
+          <mesh filename="$(find mobile_manipulator_description)/meshes/d435_with_cam_stand.stl" scale="1 1 1"/>
         </geometry>
         <material name="Grey">
@@ -13,12 +13,12 @@
       </visual>
       <collision>
-        <origin xyz="0 0 0" rpy="0 0 1.57"/>
+        <origin xyz="0 0 0" rpy="1.57 3.14 1.57"/>
         <geometry>
-          <mesh filename="$(find mobile_manipulator_description)/meshes/realsense.dae" scale="1 1 1"/>
+          <mesh filename="$(find mobile_manipulator_description)/meshes/d435_with_cam_stand.stl" scale="1 1 1"/>
         </geometry>
       </collision>
       <inertial>
         <origin xyz="0 0 0" rpy="1.57 0 1.57"/>
-        <mass value="0.0615752"/>
+        <mass value="0.002"/>
         <inertia ixx="9.108e-05" ixy="0" ixz="0" iyy="2.51e-06" iyz="0" izz="8.931e-05"/>
       </inertial>

File: MOBILE_MANIPULATOR/mobile_manipulator_description/urdf/mobile_manipulator.urdf.xacro (robot description, xacro)
@@ -2,16 +2,10 @@
 <robot name="mobile_manipulator" xmlns:xacro="http://www.ros.org/wiki/xacro">
   <xacro:include filename="$(find alphabot_description)/urdf/alphabot.urdf.xacro"/>
-  <xacro:include filename="$(find mobile_manipulator_description)/urdf/linear_guide.xacro"/>
   <xacro:include filename="$(find rm_description)/urdf/rm_75_gazebo.urdf"/>
   <xacro:include filename="$(find mobile_manipulator_description)/urdf/mobile_manipulator_ros_contol.xacro"/>
-  <joint name="chassis_to_column" type="fixed">
+  <joint name="chassis_link_to_arm_base" type="fixed">
     <parent link="chassis_link"/>
-    <child  link="column"/>
-    <origin xyz="0 0 0.1" rpy="0 0 1.57"/>
-  </joint>
-  <joint name="slider_to_arm_base" type="fixed">
-    <parent link="slider"/>
     <child  link="base_link"/>
-    <origin xyz="0 -0.33 0.06" rpy="0 0 0"/>
+    <origin xyz="0 0.1 0.4" rpy="0 0 -1.57"/>
   </joint>
   <gazebo>
@@ -38,36 +32,12 @@
     </gazebo>
   <xacro:include filename="$(find mobile_manipulator_description)/urdf/camera_module.urdf.xacro"/>
-  <link name="cylinder_link">
-  <visual>
-    <geometry>
-      <cylinder radius="0.01" length="0.71"/>
-    </geometry>
-    <material name="Grey">
-      <color rgba="0.7 0.7 0.7 1"/>
-    </material>
-  </visual>
-  <collision>
-    <geometry>
-      <cylinder radius="0.01" length="0.71"/>
-    </geometry>
-  </collision>
-  <inertial>
-    <mass value="0.5"/>
-    <inertia ixx="0.001" ixy="0" ixz="0" iyy="0.001" iyz="0" izz="0.001"/>
-  </inertial>
-</link>
- <joint name="rod_to_camera" type="fixed">
-    <parent link="camera_link_base"/>
-    <child  link="cylinder_link"/>
-    <origin xyz="0.01 0 -0.36" rpy="0 0 0"/>
-  </joint>
-    <gazebo reference="cylinder_link">
-      <material>Gazebo/Grey</material>
+      <gazebo reference="camera_link_base">
+      <material>Gazebo/Orange</material>
   </gazebo>
   <xacro:intel_d435_camera/>
   <joint name="sliderto_camera" type="fixed">
-    <parent link="link_base"/>
+    <parent link="Link7"/>
     <child  link="camera_link_base"/>
-    <origin xyz="-0.3 0.3 0.85" rpy="0 0 0"/>
+    <origin xyz="0 0 0" rpy="0 -1.57 -1.57"/>
   </joint>
 </robot>

File: REALMAN_7DOF/rm_description/urdf/rm_75_gazebo.urdf (robot description, URDF)
Before this commit: robot rm_75_description, 8 links, 7 joints
Links:
- added link tool0, mass 0.001; collision mesh filename=file://$(find rm_description)/meshes/rm_75_arm/object.stl scale=0.001 0.001 0.001; visual mesh filename=file://$(find rm_description)/meshes/rm_75_arm/object.stl scale=0.001 0.001 0.001
Joints:
- added joint joint_tool0: type fixed, parent Link7, child tool0, origin xyz=0 0 0.15 rpy=0 0 1.57

Commit message: Added vision and picking node

File: MOBILE_MANIPULATOR/mobile_manipulator_description/urdf/camera_module.urdf.xacro (robot description, xacro)
@@ -4,7 +4,7 @@
     <link name="camera_link_base">
       <visual>
-        <origin xyz="0 0 0" rpy="1.57 3.14 1.57"/>
+        <origin xyz="0 0 0" rpy="0.57 0 1.57"/>
         <geometry>
-          <mesh filename="$(find mobile_manipulator_description)/meshes/d435_with_cam_stand.stl" scale="1 1 1"/>
+          <mesh filename="$(find mobile_manipulator_description)/meshes/realsense.dae" scale="1 1 1"/>
         </geometry>
         <material name="Grey">
@@ -13,12 +13,12 @@
       </visual>
       <collision>
-        <origin xyz="0 0 0" rpy="1.57 3.14 1.57"/>
+        <origin xyz="0 0 0" rpy="0.57 0 1.57"/>
         <geometry>
-          <mesh filename="$(find mobile_manipulator_description)/meshes/d435_with_cam_stand.stl" scale="1 1 1"/>
+          <mesh filename="$(find mobile_manipulator_description)/meshes/realsense.dae" scale="1 1 1"/>
         </geometry>
       </collision>
       <inertial>
         <origin xyz="0 0 0" rpy="1.57 0 1.57"/>
-        <mass value="0.002"/>
+        <mass value="0.0615752"/>
         <inertia ixx="9.108e-05" ixy="0" ixz="0" iyy="2.51e-06" iyz="0" izz="8.931e-05"/>
       </inertial>
@@ -28,5 +28,5 @@
       <parent link="camera_link_base"/>
       <child link="camera_rgb_link"/>
-      <origin xyz="0 0 0" rpy="0 0 0"/>
+      <origin xyz="0 0 0" rpy="0 0.57 0"/>
     </joint>
     <link name="camera_rgb_optical_frame"/>
@@ -66,5 +66,5 @@
       <parent link="camera_link_base"/>
       <child link="camera_depth_link"/>
-      <origin xyz="0 0 0" rpy="0 0 0"/>
+      <origin xyz="0 0 0" rpy="0 0.57 0"/>
     </joint>
     <link name="camera_depth_optical_frame"/>
@@ -83,5 +83,5 @@
             <width>640</width>
             <height>480</height>
-            <format>DEPTH16</format>
+            <format>R8G8B8</format>
           </image>
           <clip>

File: MOBILE_MANIPULATOR/mobile_manipulator_description/urdf/linear_guide.xacro (robot description, xacro)
@@ -49,8 +49,8 @@
       <material>Gazebo/Grey</material>
   </gazebo>
-  <joint name="slider_joint" type="prismatic">
+  <joint name="slider_joint" type="fixed">
     <parent link="column"/>
     <child link="slider"/>
-    <origin xyz="0 0 0" rpy="0 0 0"/>
+    <origin xyz="0 0 0.3" rpy="0 0 0"/>
     <axis xyz="0 0 1"/>
     <limit lower="0.0" upper="0.9" effort="200" velocity="0.3"/>

File: MOBILE_MANIPULATOR/mobile_manipulator_description/urdf/mobile_manipulator.urdf.xacro (robot description, xacro)
@@ -2,10 +2,16 @@
 <robot name="mobile_manipulator" xmlns:xacro="http://www.ros.org/wiki/xacro">
   <xacro:include filename="$(find alphabot_description)/urdf/alphabot.urdf.xacro"/>
+  <xacro:include filename="$(find mobile_manipulator_description)/urdf/linear_guide.xacro"/>
   <xacro:include filename="$(find rm_description)/urdf/rm_75_gazebo.urdf"/>
   <xacro:include filename="$(find mobile_manipulator_description)/urdf/mobile_manipulator_ros_contol.xacro"/>
-  <joint name="chassis_link_to_arm_base" type="fixed">
+  <joint name="chassis_to_column" type="fixed">
     <parent link="chassis_link"/>
+    <child  link="column"/>
+    <origin xyz="0.2 -0.1 0.1" rpy="0 0 -1.57"/>
+  </joint>
+  <joint name="slider_to_arm_base" type="fixed">
+    <parent link="slider"/>
     <child  link="base_link"/>
-    <origin xyz="0 -0.2 0.5" rpy="0 0 -1.57"/>
+    <origin xyz="0 -0.33 0.06" rpy="0 0 0"/>
   </joint>
   <gazebo>
@@ -32,12 +38,36 @@
     </gazebo>
   <xacro:include filename="$(find mobile_manipulator_description)/urdf/camera_module.urdf.xacro"/>
-      <gazebo reference="camera_link_base">
-      <material>Gazebo/Orange</material>
+  <link name="cylinder_link">
+  <visual>
+    <geometry>
+      <cylinder radius="0.01" length="0.71"/>
+    </geometry>
+    <material name="Grey">
+      <color rgba="0.7 0.7 0.7 1"/>
+    </material>
+  </visual>
+  <collision>
+    <geometry>
+      <cylinder radius="0.01" length="0.71"/>
+    </geometry>
+  </collision>
+  <inertial>
+    <mass value="0.5"/>
+    <inertia ixx="0.001" ixy="0" ixz="0" iyy="0.001" iyz="0" izz="0.001"/>
+  </inertial>
+</link>
+ <joint name="rod_to_camera" type="fixed">
+    <parent link="camera_link_base"/>
+    <child  link="cylinder_link"/>
+    <origin xyz="-0.01 0 -0.36" rpy="0 0 0"/>
+  </joint>
+    <gazebo reference="cylinder_link">
+      <material>Gazebo/Grey</material>
   </gazebo>
   <xacro:intel_d435_camera/>
   <joint name="sliderto_camera" type="fixed">
-    <parent link="Link7"/>
+    <parent link="link_base"/>
     <child  link="camera_link_base"/>
-    <origin xyz="0 0 0" rpy="0 -1.57 -1.57"/>
+    <origin xyz="-0.3 0.1 1.0" rpy="0 0 -1.57"/>
   </joint>
 </robot>

File: MOBILE_MANIPULATOR/mobile_manipulator_description/urdf/mobile_manipulator_ros_contol.xacro (robot description, xacro)
@@ -5,9 +5,9 @@
       <plugin>gazebo_ros2_control/GazeboSystem</plugin>
     </hardware>
-    <joint name="slider_joint">
+    <!-- <joint name="slider_joint">
       <command_interface name="position"/>
       <state_interface name="position"/>
       <state_interface name="velocity"/>
-    </joint>
+    </joint> -->
     <joint name="joint1">
       <command_interface name="position"/>
@@ -46,5 +46,5 @@
     </joint>
   </ros2_control>
-  <transmission name="slider_trans">
+  <!-- <transmission name="slider_trans">
     <type>transmission_interface/SimpleTransmission</type>
     <joint name="slider_joint">
@@ -55,5 +55,5 @@
       <mechanicalReduction>1</mechanicalReduction>
     </actuator>
-  </transmission>
+  </transmission> -->
   <transmission name="joint1_trans">
     <type>transmission_interface/SimpleTransmission</type>
