Commit message: Refactored urdf

File: MOBILE_MANIPULATOR/mobile_manipulator_description/urdf/linear_guide.xacro (robot description, xacro)
@@ -28,5 +28,5 @@
     <visual>
       <geometry>
-        <box size="0.3 0.3 0.05"/>
+        <box size="0.25 0.25 0.05"/>
       </geometry>
       <origin xyz="0 -0.25 0.05" rpy="0 0 0"/>
@@ -37,5 +37,5 @@
     <collision>
       <geometry>
-        <box size="0.3 0.3 0.05"/>
+        <box size="0.25 0.25 0.05"/>
       </geometry>
       <origin xyz="0 -0.25 0.05" rpy="0 0 0"/>
@@ -52,5 +52,5 @@
     <parent link="column"/>
     <child link="slider"/>
-    <origin xyz="0 0 0.3" rpy="0 0 0"/>
+    <origin xyz="0 0 0.45" rpy="0 0 0"/>
     <axis xyz="0 0 1"/>
     <limit lower="0.0" upper="0.9" effort="200" velocity="0.3"/>

File: REALMAN_7DOF/rm_description/urdf/rm_75.urdf (robot description, URDF)
Before this commit: robot rm_75_description, 9 links, 8 joints
Joints:
- joint joint_tool0: origin xyz=0 0 0.13 rpy=0 0 1.57 -> xyz=0 0 0.1 rpy=0 0 1.57

File: REALMAN_7DOF/rm_description/urdf/rm_75_gazebo.urdf (robot description, URDF)
Before this commit: robot rm_75_description, 9 links, 8 joints
Joints:
- joint joint_tool0: origin xyz=0 0 0.13 rpy=0 0 1.57 -> xyz=0 0 0.1 rpy=0 0 1.57
