Commit message: Added models for gazebo

File: MOBILE_MANIPULATOR/mobile_manipulator_description/urdf/mobile_manipulator.urdf.xacro (robot description, xacro)
@@ -7,5 +7,5 @@
     <parent link="chassis_link"/>
     <child  link="base_link"/>
-    <origin xyz="0 0.1 0.4" rpy="0 0 -1.57"/>
+    <origin xyz="0 -0.2 0.5" rpy="0 0 -1.57"/>
   </joint>
   <gazebo>

File: REALMAN_7DOF/rm_description/urdf/rm_75.urdf (robot description, URDF)
Before this commit: robot rm_75_description, 9 links, 8 joints
Joints:
- joint joint_tool0: origin xyz=0 0 0.1 rpy=0 0 1.57 -> xyz=0 0 0.13 rpy=0 0 1.57

File: REALMAN_7DOF/rm_description/urdf/rm_75_gazebo.urdf (robot description, URDF)
Before this commit: robot rm_75_description, 9 links, 8 joints
Joints:
- joint joint_tool0: origin xyz=0 0 0.15 rpy=0 0 1.57 -> xyz=0 0 0.13 rpy=0 0 1.57

Commit message: Fix joint origin in mobile manipulator URDF and add AttachDetach service client in pick controller

File: MOBILE_MANIPULATOR/mobile_manipulator_description/urdf/mobile_manipulator.urdf.xacro (robot description, xacro)
@@ -13,5 +13,5 @@
     <parent link="slider"/>
     <child  link="base_link"/>
-    <origin xyz="0 -0.33 0.06" rpy="0 0 0"/>
+    <origin xyz="0 -0.33 0.04" rpy="0 0 0"/>
   </joint>
   <gazebo>
