Commit message: Refactor mobile manipulator and vision components
- Updated mass values for linear guide components in URDF to a more realistic value.
- Commented out the box_link definition in mobile manipulator URDF for future reference.
- Adjusted the position of the camera joint in the mobile manipulator URDF.
- Enhanced README with ROS 2 commands for controlling the robot and conveyor.
- Scaled mesh files in the REALMAN 7DOF URDF to improve visual representation.
- Modified box spawner plugin to spawn boxes at a new fixed position.
- Improved pick controller to include dynamic parameters and refined grasping logic.
- Updated vision node to include ArUco marker parameters for better tracking.

File: ALPHA_BOT/alphabot_description/urdf/alphabot.urdf.xacro (robot description, xacro)
@@ -47,5 +47,5 @@
         <parent link="base_footprint"/>
         <child link="link_base"/>
-        <origin xyz="0 0 ${chassis_height/2 + traction_wheel_radius}" rpy="0 0 1.57" />
+        <origin xyz="1.035312 3.917791 ${chassis_height/2 + traction_wheel_radius}" rpy="0 0 1.57" />
     </joint>
     <link name="chassis_link">

File: MOBILE_MANIPULATOR/mobile_manipulator_description/urdf/linear_guide.xacro (robot description, xacro)
@@ -18,5 +18,5 @@
     </collision>
     <inertial>
-      <mass value="5.0"/>
+      <mass value="0.0001"/>
       <inertia ixx="0.1" iyy="0.1" izz="0.1" ixy="0.0" ixz="0.0" iyz="0.0"/>
     </inertial>
@@ -42,5 +42,5 @@
     </collision>
     <inertial>
-      <mass value="2.0"/>
+      <mass value="0.0001"/>
       <inertia ixx="0.1" iyy="0.1" izz="0.1" ixy="0.0" ixz="0.0" iyz="0.0"/>
     </inertial>

File: MOBILE_MANIPULATOR/mobile_manipulator_description/urdf/mobile_manipulator.urdf.xacro (robot description, xacro)
@@ -62,4 +62,29 @@
     <origin xyz="-0.01 0 -0.36" rpy="0 0 0"/>
   </joint>
+  <!-- <link name="box_link">
+  <visual>
+    <geometry>
+      <box size="0.087220 0.116244 0.776193"/>
+    </geometry>
+    <material name="Grey">
+      <color rgba="0.7 0.7 0.7 1"/>
+    </material>
+  </visual>
+  <collision>
+    <geometry>
+      <box size="0.087220 0.116244 0.776193"/>
+    </geometry>
+  </collision>
+  <inertial>
+    <mass value="10.0"/>
+    <inertia ixx="0.001" ixy="0" ixz="0" iyy="0.001" iyz="0" izz="0.001"/>
+  </inertial>
+</link>
+ <joint name="box_linkto_linkbase" type="fixed">
+    <parent link="link_base"/>
+    <child  link="box_link"/>
+    <origin xyz="0 0.1 0.5" rpy="0 1.57 0"/>
+  </joint>
+ -->
     <gazebo reference="cylinder_link">
       <material>Gazebo/Grey</material>
@@ -69,5 +94,5 @@
     <parent link="link_base"/>
     <child  link="camera_link_base"/>
-    <origin xyz="-0.3 0.1 1.0" rpy="0 0 -1.57"/>
+    <origin xyz="-0.3 0.18 1.0" rpy="0 0 -1.57"/>
   </joint>
 </robot>

File: REALMAN_7DOF/rm_description/urdf/rm_75.urdf (robot description, URDF)
Before this commit: robot rm_75_description, 9 links, 8 joints
Links:
- link Link1: geometry collision mesh filename=package://rm_description/meshes/rm_75_arm/link1.STL scale=1.5 1.5 1.5; visual mesh filename=package://rm_description/meshes/rm_75_arm/link1.STL scale=1.5 1.5 1.5
- link Link2: geometry collision mesh filename=package://rm_description/meshes/rm_75_arm/link2.STL scale=1.5 1.5 1.5; visual mesh filename=package://rm_description/meshes/rm_75_arm/link2.STL scale=1.5 1.5 1.5
- link Link3: geometry collision mesh filename=package://rm_description/meshes/rm_75_arm/link3.STL scale=1.5 1.5 1.5; visual mesh filename=package://rm_description/meshes/rm_75_arm/link3.STL scale=1.5 1.5 1.5
- link Link4: geometry collision mesh filename=package://rm_description/meshes/rm_75_arm/link4.STL scale=1.5 1.5 1.5; visual mesh filename=package://rm_description/meshes/rm_75_arm/link4.STL scale=1.5 1.5 1.5
- link Link5: geometry collision mesh filename=package://rm_description/meshes/rm_75_arm/link5.STL scale=1.5 1.5 1.5; visual mesh filename=package://rm_description/meshes/rm_75_arm/link5.STL scale=1.5 1.5 1.5
- link Link6: geometry collision mesh filename=package://rm_description/meshes/rm_75_arm/link6.STL scale=1.5 1.5 1.5; visual mesh filename=package://rm_description/meshes/rm_75_arm/link6.STL scale=1.5 1.5 1.5
- link Link7: geometry collision mesh filename=package://rm_description/meshes/rm_75_arm/link7.STL scale=1.5 1.5 1.5; visual mesh filename=package://rm_description/meshes/rm_75_arm/link7.STL scale=1.5 1.5 1.5
- link base_link: geometry collision mesh filename=package://rm_description/meshes/rm_75_arm/base_link.STL scale=1.5 1.5 1.5; visual mesh filename=package://rm_description/meshes/rm_75_arm/base_link.STL scale=1.5 1.5 1.5
- link tool0: geometry collision mesh filename=file://$(find rm_description)/meshes/rm_75_arm/object.stl scale=0.0015 0.0015 0.0015; visual mesh filename=file://$(find rm_description)/meshes/rm_75_arm/object.stl scale=0.0015 0.0015 0.0015
Joints:
- joint joint1: origin xyz=0 0 0.2405 rpy=-1.5708 0 0 -> xyz=0 0 0.36075 rpy=-1.5708 0 0
- joint joint3: origin xyz=0 0 0.256 rpy=-1.5708 0 0 -> xyz=0 0 0.384 rpy=-1.5708 0 0
- joint joint5: origin xyz=0 0 0.21 rpy=-1.5708 0 0 -> xyz=0 0 0.315 rpy=-1.5708 0 0
- joint joint7: origin xyz=0 0 0.144 rpy=0 0 0 -> xyz=0 0 0.216 rpy=0 0 0
- joint joint_tool0: origin xyz=0 0 0.1 rpy=0 0 1.57 -> xyz=0 0 0.15 rpy=0 0 1.57

File: REALMAN_7DOF/rm_description/urdf/rm_75_gazebo.urdf (robot description, URDF)
Before this commit: robot rm_75_description, 9 links, 8 joints
Links:
- link Link1: geometry collision mesh filename=file://$(find rm_description)/meshes/rm_75_arm/link1.STL scale=1.5 1.5 1.5; visual mesh filename=file://$(find rm_description)/meshes/rm_75_arm/link1.STL scale=1.5 1.5 1.5
- link Link2: geometry collision mesh filename=file://$(find rm_description)/meshes/rm_75_arm/link2.STL scale=1.5 1.5 1.5; visual mesh filename=file://$(find rm_description)/meshes/rm_75_arm/link2.STL scale=1.5 1.5 1.5
- link Link3: geometry collision mesh filename=file://$(find rm_description)/meshes/rm_75_arm/link3.STL scale=1.5 1.5 1.5; visual mesh filename=file://$(find rm_description)/meshes/rm_75_arm/link3.STL scale=1.5 1.5 1.5
- link Link4: geometry collision mesh filename=file://$(find rm_description)/meshes/rm_75_arm/link4.STL scale=1.5 1.5 1.5; visual mesh filename=file://$(find rm_description)/meshes/rm_75_arm/link4.STL scale=1.5 1.5 1.5
- link Link5: geometry collision mesh filename=file://$(find rm_description)/meshes/rm_75_arm/link5.STL scale=1.5 1.5 1.5; visual mesh filename=file://$(find rm_description)/meshes/rm_75_arm/link5.STL scale=1.5 1.5 1.5
- link Link6: geometry collision mesh filename=file://$(find rm_description)/meshes/rm_75_arm/link6.STL scale=1.5 1.5 1.5; visual mesh filename=file://$(find rm_description)/meshes/rm_75_arm/link6.STL scale=1.5 1.5 1.5
- link Link7: geometry collision mesh filename=file://$(find rm_description)/meshes/rm_75_arm/link7.STL scale=1.5 1.5 1.5; visual mesh filename=file://$(find rm_description)/meshes/rm_75_arm/link7.STL scale=1.5 1.5 1.5
- link base_link: geometry collision mesh filename=file://$(find rm_description)/meshes/rm_75_arm/base_link.STL scale=1.5 1.5 1.5; visual mesh filename=file://$(find rm_description)/meshes/rm_75_arm/base_link.STL scale=1.5 1.5 1.5
- link tool0: mass 0.001 -> 0.1; geometry collision mesh filename=file://$(find rm_description)/meshes/rm_75_arm/object.stl scale=0.0015 0.0015 0.0015; visual mesh filename=file://$(find rm_description)/meshes/rm_75_arm/object.stl scale=0.0015 0.0015 0.0015
Joints:
- joint joint1: origin xyz=0 0 0.2405 rpy=-1.5708 0 0 -> xyz=0 0 0.36075 rpy=-1.5708 0 0
- joint joint3: origin xyz=0 0 0.256 rpy=-1.5708 0 0 -> xyz=0 0 0.384 rpy=-1.5708 0 0
- joint joint5: origin xyz=0 0 0.21 rpy=-1.5708 0 0 -> xyz=0 0 0.315 rpy=-1.5708 0 0
- joint joint7: origin xyz=0 0 0.144 rpy=0 0 0 -> xyz=0 0 0.216 rpy=0 0 0
- joint joint_tool0: origin xyz=0 0 0.1 rpy=0 0 1.57 -> xyz=0 0 0.15 rpy=0 0 1.57
